File: PCBs/LabelModule/Label/Label.sch (KiCad schematic (older format))
At the start: 10 parts

Commit message: This advancement creates the schematics to drive the screen. Next part is to add other required modules and start designing the PCB
Parts:
- added C? (x2): 50 v 1 uF, Capacitor_SMD:C_0201_0603Metric, symbol Device:C
- added C? (x3): 50 V 1uF, Capacitor_SMD:C_0201_0603Metric, symbol Device:C
- added C? (x6): 25 V 1uF, Capacitor_SMD:C_0201_0603Metric, symbol Device:C
- added CONN?: CrystalFontz24-pinCFAP-ePaper, symbol CrystalFontz:CrystalFontz24-pinCFAP-ePaper
- added D? (x3): MBR0530, Diode_SMD:D_SOD-123, symbol Diode:MBR0530
- added L?: COILCRAFT LPS3015-140MRC 3.4 OHM, 100 uH 240 mA, symbol Device:L
- added Q?: IRLML6346TRPBF, Package_TO_SOT_SMD:TSOT-23, symbol Transistor_FET:DMC3071LVT
- added R?: 0.47 1%, Resistor_SMD:R_0603_1608Metric, symbol Device:R
- added R?: 100K, Resistor_SMD:R_0603_1608Metric, symbol Device:R
- added U?: RC-CC1310R-XXX, symbol Radiocontrolli:RC-CC1310R-XXX
- R?: value 1.87MOhm -> 1.1Mohm
Connections:
- net GND: now also C?.1, C?.2, C?.2, C?.2, C?.2, C?.2, C?.2, C?.2, C?.2, C?.2, CONN?.17 (VSS), CONN?.8 (BS1), D?.1 (K), R?.2, R?.2, U?.1 (GND), U?.9 (GND)
- net +3V3: now reaches C?.1, C?.1, R?.1, U?.1*3 (VOUT)
- net +3V3: now also C?.1, CONN?.15 (VDDIO), CONN?.16 (VCI), L?.1, U?.10 (VDD)
- net +BATT: now reaches C?.1, C?.1, L?.1, R?.1, U?.8 (VBAT)
- new net: Q?.5 (S), R?.1
- new net: C?.1, D?.2 (A), L?.2, Q?.6 (D)
- new net: C?.1, CONN?.18 (VDD)
- new net: C?.1, CONN?.19 (VPP)
- new net: C?.1, CONN?.20 (VSH)
- new net: C?.1, CONN?.22 (VSL)
- new net: C?.1, CONN?.24 (VCOM)
- new net: C?.1, CONN?.4 (VGL)
- new net: C?.1, CONN?.5 (VGH)
- new net BUSY: CONN?.9 (BUSY), U?.17 (DIO-14)
- new net DC: U?.15 (DIO-12)
- new net D~C: CONN?.11 (D/~C)
- new net GDR: CONN?.2 (GDR), Q?.1 (G), R?.1
- new net GNDPWR: CONN?.25 (CONPAD), CONN?.26 (CONPAD)
- new net MOSI: CONN?.14 (D1(MOSI)), U?.12 (DIO-9)
- new net PREVGH: C?.1, CONN?.21 (PREVHG), D?.1 (K)
- new net PREVGL: C?.2, CONN?.23 (PREVGL), D?.2 (A)
- new net RESE: C?.2, CONN?.3 (RESE), D?.1 (K), D?.2 (A)
- new net SCK: CONN?.13 (D0(SCK)), U?.13 (DIO-10)
- new net ~CS: CONN?.12 (~CS), U?.14 (DIO-11)
- new net ~RST: CONN?.10 (~RST), U?.16 (DIO-13)
- no-connect marks 0 -> 3
Other:
- moved on the sheet: C?, L?, R?, U?
